Commit message: 1.2gazebo

File: src/cakebot_description/urdf/cakebot.urdf.xacro (robot description, xacro)
@@ -6,6 +6,7 @@
     y：机器人左方为正，右方为负
     z：向上为正
-  本文件刻意把几何尺寸和组件位置集中在顶部，方便在实物尺寸尚未
-  完全确定时调整。当前模型用于 RViz 显示，暂不包含 Gazebo 插件。
+  本文件刻意把几何尺寸、质量和组件位置集中在顶部，方便在实物尺寸
+  尚未完全确定时调整。模型包含可用于 Gazebo 的 visual、collision 和
+  inertial 数据；差速驱动、传感器等功能由后续阶段单独加入。
 -->
 <robot xmlns:xacro="http://www.ros.org/wiki/xacro" name="cakebot">
@@ -26,4 +27,5 @@
   <xacro:arg name="wheel_z" default="0.05"/>
   <xacro:arg name="wheel_mass" default="0.15"/>
+  <xacro:arg name="wheel_damping" default="0.01"/>
   <!--
     万向轮位置：
@@ -54,4 +56,5 @@
   <xacro:property name="wheel_z" value="$(arg wheel_z)"/>
   <xacro:property name="wheel_mass" value="$(arg wheel_mass)"/>
+  <xacro:property name="wheel_damping" value="$(arg wheel_damping)"/>
   <xacro:property name="caster_radius" value="$(arg caster_radius)"/>
   <xacro:property name="caster_x" value="$(arg caster_x)"/>
@@ -77,7 +80,8 @@
     </inertial>
   </xacro:macro>
-  <!-- 圆柱惯性：宏内部默认圆柱轴线为 z 轴 -->
-  <xacro:macro name="cylinder_inertial" params="mass radius length">
+  <!-- 圆柱惯性：宏内部默认圆柱轴线为 z 轴。 -->
+  <xacro:macro name="cylinder_inertial" params="mass radius length origin_rpy">
     <inertial>
+      <origin xyz="0 0 0" rpy="${origin_rpy}"/>
       <mass value="${mass}"/>
       <inertia
@@ -88,4 +92,18 @@
         iyz="0.0"
         izz="${mass * radius * radius / 2.0}"/>
+    </inertial>
+  </xacro:macro>
+  <!-- 球体惯性。球体的质心位于 link 原点。 -->
+  <xacro:macro name="sphere_inertial" params="mass radius">
+    <inertial>
+      <origin xyz="0 0 0" rpy="0 0 0"/>
+      <mass value="${mass}"/>
+      <inertia
+        ixx="${2.0 * mass * radius * radius / 5.0}"
+        ixy="0.0"
+        ixz="0.0"
+        iyy="${2.0 * mass * radius * radius / 5.0}"
+        iyz="0.0"
+        izz="${2.0 * mass * radius * radius / 5.0}"/>
     </inertial>
   </xacro:macro>
@@ -107,15 +125,9 @@
       </collision>
       <!-- 惯性坐标系随圆柱一起绕 x 轴旋转，使圆柱轴线为 y 轴。 -->
-      <inertial>
-        <origin xyz="0 0 0" rpy="${pi / 2.0} 0 0"/>
-        <mass value="${wheel_mass}"/>
-        <inertia
-          ixx="${wheel_mass * (3.0 * wheel_radius * wheel_radius + wheel_width * wheel_width) / 12.0}"
-          ixy="0.0"
-          ixz="0.0"
-          iyy="${wheel_mass * wheel_radius * wheel_radius / 2.0}"
-          iyz="0.0"
-          izz="${wheel_mass * (3.0 * wheel_radius * wheel_radius + wheel_width * wheel_width) / 12.0}"/>
-      </inertial>
+      <xacro:cylinder_inertial
+        mass="${wheel_mass}"
+        radius="${wheel_radius}"
+        length="${wheel_width}"
+        origin_rpy="${pi / 2.0} 0 0"/>
     </link>
     <joint name="${side}_wheel_joint" type="continuous">
@@ -124,4 +136,5 @@
       <origin xyz="${wheel_x} ${y} ${wheel_z}" rpy="0 0 0"/>
       <axis xyz="0 1 0"/>
+      <dynamics damping="${wheel_damping}" friction="0.0"/>
     </joint>
   </xacro:macro>
@@ -168,5 +181,6 @@
     简化万向轮：当前使用球体表示，采用 fixed joint。
     caster_x/caster_y/caster_z/caster_yaw 均可直接调整。
-    后续进入 Gazebo 阶段时，再替换为真实的转向结构和碰撞参数。
+    当前用简化球体保证仿真模型闭合；实物尺寸确定后，再替换为真实
+    的万向轮支架和碰撞几何。
   -->
   <link name="caster_link">
@@ -184,14 +198,5 @@
       </geometry>
     </collision>
-    <inertial>
-      <mass value="${caster_mass}"/>
-      <inertia
-        ixx="${2.0 * caster_mass * caster_radius * caster_radius / 5.0}"
-        ixy="0.0"
-        ixz="0.0"
-        iyy="${2.0 * caster_mass * caster_radius * caster_radius / 5.0}"
-        iyz="0.0"
-        izz="${2.0 * caster_mass * caster_radius * caster_radius / 5.0}"/>
-    </inertial>
+    <xacro:sphere_inertial mass="${caster_mass}" radius="${caster_radius}"/>
   </link>
   <joint name="caster_joint" type="fixed">

Commit message: 激光雷达

File: src/cakebot_description/urdf/cakebot.urdf.xacro (robot description, xacro)
@@ -41,4 +41,19 @@
   <xacro:arg name="caster_yaw" default="0.0"/>
   <xacro:arg name="caster_mass" default="0.08"/>
+  <!-- 激光雷达尺寸与安装位置 -->
+  <xacro:arg name="laser_radius" default="0.035"/>
+  <xacro:arg name="laser_height" default="0.04"/>
+  <xacro:arg name="laser_x" default="0.10"/>
+  <xacro:arg name="laser_y" default="0.0"/>
+  <xacro:arg name="laser_z" default="0.17"/>
+  <xacro:arg name="laser_mass" default="0.08"/>
+  <!-- 激光雷达扫描参数 -->
+  <xacro:arg name="laser_update_rate" default="10.0"/>
+  <xacro:arg name="laser_samples" default="360"/>
+  <xacro:arg name="laser_min_angle" default="-3.14159265359"/>
+  <xacro:arg name="laser_max_angle" default="3.14159265359"/>
+  <xacro:arg name="laser_min_range" default="0.12"/>
+  <xacro:arg name="laser_max_range" default="8.0"/>
+  <xacro:arg name="laser_range_resolution" default="0.01"/>
   <!--
     将可由命令行覆盖的 xacro:arg 映射为内部属性。
@@ -63,4 +78,17 @@
   <xacro:property name="caster_yaw" value="$(arg caster_yaw)"/>
   <xacro:property name="caster_mass" value="$(arg caster_mass)"/>
+  <xacro:property name="laser_radius" value="$(arg laser_radius)"/>
+  <xacro:property name="laser_height" value="$(arg laser_height)"/>
+  <xacro:property name="laser_x" value="$(arg laser_x)"/>
+  <xacro:property name="laser_y" value="$(arg laser_y)"/>
+  <xacro:property name="laser_z" value="$(arg laser_z)"/>
+  <xacro:property name="laser_mass" value="$(arg laser_mass)"/>
+  <xacro:property name="laser_update_rate" value="$(arg laser_update_rate)"/>
+  <xacro:property name="laser_samples" value="$(arg laser_samples)"/>
+  <xacro:property name="laser_min_angle" value="$(arg laser_min_angle)"/>
+  <xacro:property name="laser_max_angle" value="$(arg laser_max_angle)"/>
+  <xacro:property name="laser_min_range" value="$(arg laser_min_range)"/>
+  <xacro:property name="laser_max_range" value="$(arg laser_max_range)"/>
+  <xacro:property name="laser_range_resolution" value="$(arg laser_range_resolution)"/>
   <!-- ================================================================
        可复用宏
@@ -151,4 +179,7 @@
     <color rgba="0.45 0.45 0.45 1.0"/>
   </material>
+  <material name="laser_black">
+    <color rgba="0.02 0.02 0.02 1.0"/>
+  </material>
   <!-- ================================================================
        机器人主体
@@ -205,4 +236,60 @@
     <origin xyz="${caster_x} ${caster_y} ${caster_z}" rpy="0 0 ${caster_yaw}"/>
   </joint>
+  <!-- 激光雷达安装座。雷达坐标系 z 轴向上，x 轴指向机器人前方。 -->
+  <link name="laser_link">
+    <visual>
+      <origin xyz="0 0 0" rpy="0 0 0"/>
+      <geometry>
+        <cylinder radius="${laser_radius}" length="${laser_height}"/>
+      </geometry>
+      <material name="laser_black"/>
+    </visual>
+    <collision>
+      <origin xyz="0 0 0" rpy="0 0 0"/>
+      <geometry>
+        <cylinder radius="${laser_radius}" length="${laser_height}"/>
+      </geometry>
+    </collision>
+    <xacro:cylinder_inertial
+      mass="${laser_mass}"
+      radius="${laser_radius}"
+      length="${laser_height}"
+      origin_rpy="0 0 0"/>
+  </link>
+  <joint name="laser_joint" type="fixed">
+    <parent link="base_link"/>
+    <child link="laser_link"/>
+    <origin xyz="${laser_x} ${laser_y} ${laser_z}" rpy="0 0 0"/>
+  </joint>
+  <!-- Gazebo Classic 激光雷达传感器。扫描结果由 gazebo_ros 发布到 /scan。 -->
+  <gazebo reference="laser_link">
+    <sensor name="cakebot_laser" type="ray">
+      <pose>0 0 0 0 0 0</pose>
+      <visualize>true</visualize>
+      <update_rate>${laser_update_rate}</update_rate>
+      <ray>
+        <scan>
+          <horizontal>
+            <samples>${laser_samples}</samples>
+            <resolution>1</resolution>
+            <min_angle>${laser_min_angle}</min_angle>
+            <max_angle>${laser_max_angle}</max_angle>
+          </horizontal>
+        </scan>
+        <range>
+          <min>${laser_min_range}</min>
+          <max>${laser_max_range}</max>
+          <resolution>${laser_range_resolution}</resolution>
+        </range>
+      </ray>
+      <plugin name="cakebot_laser_sensor" filename="libgazebo_ros_ray_sensor.so">
+        <ros>
+          <remapping>~/out:=scan</remapping>
+        </ros>
+        <output_type>sensor_msgs/LaserScan</output_type>
+        <frame_name>laser_link</frame_name>
+      </plugin>
+    </sensor>
+  </gazebo>
   <!-- ================================================================
        Gazebo Classic 差速驱动插件

Commit message: 适配mid360 建图算法不用改3d但改用mid360 故3d和2d适配器

File: src/cakebot_description/urdf/cakebot.urdf.xacro (robot description, xacro)
@@ -48,4 +48,23 @@
   <xacro:arg name="laser_z" default="0.17"/>
   <xacro:arg name="laser_mass" default="0.08"/>
+  <!--
+    感知模式：
+      laser_2d  : 保留原有的二维 LaserScan 传感器；
+      mid360_sim: 使用带垂直扫描的三维仿真雷达，输出 PointCloud2。
+    两种模式只能同时启用一种，避免产生两个传感器发布同一个接口。
+  -->
+  <xacro:arg name="sensor_mode" default="laser_2d"/>
+  <!-- 是否在 Gazebo GUI 中绘制雷达射线；不影响传感器消息发布。 -->
+  <xacro:arg name="visualize_lidar" default="true"/>
+  <xacro:arg name="mid360_update_rate" default="10.0"/>
+  <xacro:arg name="mid360_horizontal_samples" default="360"/>
+  <!-- 仿真默认用 16 条垂直采样保持 Gazebo 在普通电脑上接近10 Hz；真机点云密度由驱动器决定。 -->
+  <xacro:arg name="mid360_vertical_samples" default="16"/>
+  <xacro:arg name="mid360_min_vertical_angle" default="-0.1221730476"/>
+  <xacro:arg name="mid360_max_vertical_angle" default="0.9075712110"/>
+  <xacro:arg name="mid360_min_range" default="0.10"/>
+  <xacro:arg name="mid360_max_range" default="40.0"/>
+  <xacro:arg name="mid360_range_resolution" default="0.01"/>
+  <xacro:arg name="mid360_points_topic" default="lidar/points_raw"/>
   <!-- 激光雷达扫描参数 -->
   <xacro:arg name="laser_update_rate" default="10.0"/>
@@ -84,4 +103,15 @@
   <xacro:property name="laser_z" value="$(arg laser_z)"/>
   <xacro:property name="laser_mass" value="$(arg laser_mass)"/>
+  <xacro:property name="sensor_mode" value="$(arg sensor_mode)"/>
+  <xacro:property name="visualize_lidar" value="$(arg visualize_lidar)"/>
+  <xacro:property name="mid360_update_rate" value="$(arg mid360_update_rate)"/>
+  <xacro:property name="mid360_horizontal_samples" value="$(arg mid360_horizontal_samples)"/>
+  <xacro:property name="mid360_vertical_samples" value="$(arg mid360_vertical_samples)"/>
+  <xacro:property name="mid360_min_vertical_angle" value="$(arg mid360_min_vertical_angle)"/>
+  <xacro:property name="mid360_max_vertical_angle" value="$(arg mid360_max_vertical_angle)"/>
+  <xacro:property name="mid360_min_range" value="$(arg mid360_min_range)"/>
+  <xacro:property name="mid360_max_range" value="$(arg mid360_max_range)"/>
+  <xacro:property name="mid360_range_resolution" value="$(arg mid360_range_resolution)"/>
+  <xacro:property name="mid360_points_topic" value="$(arg mid360_points_topic)"/>
   <xacro:property name="laser_update_rate" value="$(arg laser_update_rate)"/>
   <xacro:property name="laser_samples" value="$(arg laser_samples)"/>
@@ -262,34 +292,81 @@
     <origin xyz="${laser_x} ${laser_y} ${laser_z}" rpy="0 0 0"/>
   </joint>
-  <!-- Gazebo Classic 激光雷达传感器。扫描结果由 gazebo_ros 发布到 /scan。 -->
-  <gazebo reference="laser_link">
-    <sensor name="cakebot_laser" type="ray">
-      <pose>0 0 0 0 0 0</pose>
-      <visualize>true</visualize>
-      <update_rate>${laser_update_rate}</update_rate>
-      <ray>
-        <scan>
-          <horizontal>
-            <samples>${laser_samples}</samples>
-            <resolution>1</resolution>
-            <min_angle>${laser_min_angle}</min_angle>
-            <max_angle>${laser_max_angle}</max_angle>
-          </horizontal>
-        </scan>
-        <range>
-          <min>${laser_min_range}</min>
-          <max>${laser_max_range}</max>
-          <resolution>${laser_range_resolution}</resolution>
-        </range>
-      </ray>
-      <plugin name="cakebot_laser_sensor" filename="libgazebo_ros_ray_sensor.so">
-        <ros>
-          <remapping>~/out:=scan</remapping>
-        </ros>
-        <output_type>sensor_msgs/LaserScan</output_type>
-        <frame_name>laser_link</frame_name>
-      </plugin>
-    </sensor>
-  </gazebo>
+  <!--
+    Gazebo Classic 二维激光雷达。扫描结果发布到 /scan。
+    这是默认模式，用于保持阶段 5–8 的旧流程可回归。
+  -->
+  <xacro:if value="${sensor_mode == 'laser_2d'}">
+    <gazebo reference="laser_link">
+      <sensor name="cakebot_laser" type="ray">
+        <pose>0 0 0 0 0 0</pose>
+        <visualize>${visualize_lidar}</visualize>
+        <update_rate>${laser_update_rate}</update_rate>
+        <ray>
+          <scan>
+            <horizontal>
+              <samples>${laser_samples}</samples>
+              <resolution>1</resolution>
+              <min_angle>${laser_min_angle}</min_angle>
+              <max_angle>${laser_max_angle}</max_angle>
+            </horizontal>
+          </scan>
+          <range>
+            <min>${laser_min_range}</min>
+            <max>${laser_max_range}</max>
+            <resolution>${laser_range_resolution}</resolution>
+          </range>
+        </ray>
+        <plugin name="cakebot_laser_sensor" filename="libgazebo_ros_ray_sensor.so">
+          <ros>
+            <remapping>~/out:=scan</remapping>
+          </ros>
+          <output_type>sensor_msgs/LaserScan</output_type>
+          <frame_name>laser_link</frame_name>
+        </plugin>
+      </sensor>
+    </gazebo>
+  </xacro:if>
+  <!--
+    Gazebo Classic MID-360 近似仿真：水平 360 度、垂直 -7 度到 52 度。
+    输出为 sensor_msgs/PointCloud2，供 cakebot_perception 转换为 /scan。
+    这个模式不直接发布 /scan，避免与点云适配器重复。
+  -->
+  <xacro:if value="${sensor_mode == 'mid360_sim'}">
+    <gazebo reference="laser_link">
+      <sensor name="cakebot_mid360" type="ray">
+        <pose>0 0 0 0 0 0</pose>
+        <visualize>${visualize_lidar}</visualize>
+        <update_rate>${mid360_update_rate}</update_rate>
+        <ray>
+          <scan>
+            <horizontal>
+              <samples>${mid360_horizontal_samples}</samples>
+              <resolution>1</resolution>
+              <min_angle>-3.14159265359</min_angle>
+              <max_angle>3.14159265359</max_angle>
+            </horizontal>
+            <vertical>
+              <samples>${mid360_vertical_samples}</samples>
+              <resolution>1</resolution>
+              <min_angle>${mid360_min_vertical_angle}</min_angle>
+              <max_angle>${mid360_max_vertical_angle}</max_angle>
+            </vertical>
+          </scan>
+          <range>
+            <min>${mid360_min_range}</min>
+            <max>${mid360_max_range}</max>
+            <resolution>${mid360_range_resolution}</resolution>
+          </range>
+        </ray>
+        <plugin name="cakebot_mid360_sensor" filename="libgazebo_ros_ray_sensor.so">
+          <ros>
+            <remapping>~/out:=${mid360_points_topic}</remapping>
+          </ros>
+          <output_type>sensor_msgs/PointCloud2</output_type>
+          <frame_name>laser_link</frame_name>
+        </plugin>
+      </sensor>
+    </gazebo>
+  </xacro:if>
   <!-- ================================================================
        Gazebo Classic 差速驱动插件
